File: First_try.kicad_sch (KiCad schematic)
At the start: 106 parts, among them IC1 AT25FF081A-SSHN-B, IC2 ICE5LP2K-SG48ITR, J1 TYPE-611-T3-W, J5 Conn_01x20, J6 Conn_01x20, Q1 Q_NMOS_GSD, SW1 SW_Push, SW2 SW_Push, SW3 SW_Push, SW4 SW_Push, SW5 SW_Push, U1 FT232HL-REEL, U2 MCP1804x-2502xOT, U3 SN74AUP2G125DCUR, U4 INA226AIDGSR, U5 INA226AIDGSR

Commit message: LEDs, Switches
Parts:
- removed LED1, LED2, LED3: XL-1608UWC-04, LED_XL-1608_XLG, symbol WHITE_LED:XL-1608UWC-04
- removed PMOD: Conn_02x06_Odd_Even, symbol Connector_Generic:Conn_02x06_Odd_Even
- removed R23, R24: 100, symbol Device:R
- added C53: 100n, symbol Device:C
- added C54: 4.7u, symbol Device:C
- added D3, D4, D5, D6: LD274, LED_THT:LED_D5.0mm_IRGrey, symbol LED:LD274
- added D7: LED_ARBG, symbol Device:LED_ARBG
- added PMOD_OLED: Conn_02x06_Top_Bottom, symbol Connector_Generic:Conn_02x06_Top_Bottom
- added Q2, Q3, Q4, Q5: Q_NMOS_GSD, symbol Transistor_FET:Q_NMOS_GSD
- added R21, R25, R28: 10k, symbol Device:R
- added R27: 2.2k, symbol Device:R
- added R29: 121, symbol Device:R
- added R30: 158, symbol Device:R
- added R31: 115, symbol Device:R
- added R32: 162, symbol Device:R
- added R33: 70, symbol Device:R
- added R34, R35: 35, symbol Device:R
- added SW6: SW_Push, symbol Switch:SW_Push
- added SW7: EG1218, SW_1218_EWI, symbol slide_sw:EG1218
- added U6: 93LC56BT-I/OT, SOT-23-6_MC_MCH, symbol EEPROM:93LC56BT-I_OT
- R12, R7: value 200 -> 121
- R17: value 10k -> 66.5
- R8: value 100 -> 66.5
Connections:
- net FLASH_MISO is gone; now on net SDI: U1.15 (ADBUS2)
- net FLASH_MOSI is gone; now on net SDO: U1.14 (ADBUS1)
- net FT_SCK is gone; now on net SCK: U1.13 (ADBUS0)
- net FT_SSn is gone; now on net SS: U1.17 (ADBUS4)
- net +3V3: now also R8.1, C53.1, C54.1, D7.1 (A), PMOD_OLED.12 (Pin_12), PMOD_OLED.6 (Pin_6), R21.1, R25.1, R28.1, U6.6 (VCC); no longer D2.2 (A), R8.2
- net +5V: now also D2.2 (A), D3.2 (A), D4.2 (A), D5.2 (A), D6.2 (A), SW7.2; no longer C32.1, FB1.1, U1.40 (VREG)
- net EE_CLK: now also R25.2, U6.4 (CLK)
- net EE_CS: now also R21.2, U6.5 (CS)
- net EE_DAT: now also R27.1, U6.3 (DI)
- net FPGA_CLK: now also PMOD_OLED.4 (Pin_4)
- net GND: now also C53.2, C54.2, PMOD_OLED.11 (Pin_11), PMOD_OLED.5 (Pin_5), Q2.2 (S), Q3.2 (S), Q4.2 (S), Q5.2 (S), SW6.2, U6.2 (VSS)
- net SDI: now also PMOD_OLED.2 (Pin_2)
- net SS: now also PMOD_OLED.1 (Pin_1)
- net IOB_6A: now reaches IC2.2 (IOB_6A)
- net IOB_6A: now also Q2.1 (G)
- net IOB_9B: now reaches IC2.3 (IOB_9B)
- net IOB_9B: now also Q3.1 (G)
- net RES_PMOD: now reaches IC2.37 (IOT_45A_G1)
- net RES_PMOD: now also R8.2, PMOD_OLED.8 (Pin_8), SW6.1
- net DC_PMOD: now reaches IC2.38 (IOT_50B)
- net DC_PMOD: now also PMOD_OLED.7 (Pin_7)
- net IOB_8A: now reaches IC2.4 (IOB_8A)
- net IOB_8A: now also Q4.1 (G)
- net IOB_13B: now reaches IC2.6 (IOB_13B)
- net IOB_13B: now also Q5.1 (G)
- net led1 renamed R_LED
- net R_LED: now also R33.2
- net led2 renamed G_LED
- net G_LED: now also R34.2
- net led3 renamed B_LED
- net B_LED: now also R35.2
- new net: C32.1, FB1.1, SW7.1, U1.40 (VREG)
- new net: D4.1 (K), R30.1
- new net: Q3.3 (D), R30.2
- new net: R27.2, R28.2, U6.1 (DO)
- new net: D3.1 (K), R29.1
- new net: D7.4 (GK), R34.1
- new net: D7.3 (BK), R35.1
- new net: D6.1 (K), R32.1
- new net: Q5.3 (D), R32.2
- new net: Q2.3 (D), R29.2
- new net: D5.1 (K), R31.1
- new net: Q4.3 (D), R31.2
- new net: D7.2 (RK), R33.1
- no-connect marks 24 -> 19
Other:
- note added: "BLUE LED"
- note added: "C273394"
- note added: "C841777- shunt resistances"
- note added: "GREEN LED"
- note added: "NC"
- note added: "ORANGE LED"
- note added: "RED LED"
- note added: "VBAT"
- note added: "VDCC"
- moved on the sheet: C10, C24, C44, D1, D13, R1, R2, R7

Commit message: Reviewed USB-C plug
Parts:
- removed C32: 4.7u, symbol Device:C
- C27: value 100n -> 4.7u
- R6: value 330 -> 5.1k
- renumbered D7 to C22461782
Connections:
- net D_M: now also J1.B7 (DN2)
- net D_P: now also J1.B6 (DP2)
- net GND: now also C27.1, J1.A1 (GND), J1.A12 (GND), J1.B1 (GND), J1.B12 (GND), R5.1; no longer C27.2, R5.2
- net at FB1.1, SW7.1, U1.40 (VREG): now also C22.1, C27.2
- net at FB1.2, J1.A4 (VBUS), J1.A9 (VBUS)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: no longer C27.1
- net at J1.A5 (CC1): now also R5.2; no longer R5.1
- net at J1.B5 (CC2): now also R6.2
Other:
- note added: "BLUE C965807"
- note added: "GREEN C965804"
- note added: "ORANGE C965800"
- note added: "RED C965799"
- note removed: "BLUE LED"
- note removed: "GREEN LED"
- note removed: "ORANGE LED"
- note removed: "RED LED"
- moved on the sheet: FB1, R5

Commit message: Modificari dupa intalnirea de joi
Parts:
- removed J5, J6: Conn_01x20, symbol Connector_Generic:Conn_01x20
- removed R16, R19: 3.3k, symbol Device:R
- removed R26: 4.7k, symbol Device:R
- added PMOD_TMP2: Conn_02x04_Top_Bottom, symbol Connector_Generic:Conn_02x04_Top_Bottom
- R17: value 66.5 -> 10k
Connections:
- net +3V3: now also R11.1, R18.1, U5.2 (A0), PMOD_TMP2.4 (Pin_4), PMOD_TMP2.8 (Pin_8); no longer R11.2, R18.2
- net +5V: now also C27.2, U1.40 (VREG)
- net 3.3: now also C37.2, C38.2, C39.2, FB3.2, FB4.2, U1.12 (VCCIO), U1.24 (VCCIO), U1.46 (VCCIO)
- net DC_PMOD: now also IC2.43 (IOT_49A); no longer IC2.38 (IOT_50B)
- net FPGA_CLK: no longer PMOD_OLED.4 (Pin_4)
- net GND: now also PMOD_TMP2.3 (Pin_3), PMOD_TMP2.7 (Pin_7); no longer U5.2 (A0)
- net RES_PMOD: now also IC2.42 (IOT_51A); no longer IC2.37 (IOT_45A_G1)
- net SDI: now also IC1.2 (SO_(I/O1)); no longer IC1.5 (SI_(I/O0)), PMOD_OLED.2 (Pin_2)
- net SDO: now also IC1.5 (SI_(I/O0)); no longer IC1.2 (SO_(I/O1))
- net SS: no longer PMOD_OLED.1 (Pin_1)
- net at C22.1, FB1.1, SW7.1: no longer C27.2, U1.40 (VREG)
- net PMOD_CLK: now reaches IC2.44 (IOB_3B_G6)
- net PMOD_CLK: now also PMOD_OLED.4 (Pin_4)
- net 12SCL renamed SCL
- net SCL: now also R18.2, U5.5 (SCL); no longer R11.1
- net 12SDA renamed SDA
- net SDA: now also R11.2, U5.4 (SDA)
- net 33SCL renamed PMOD_SDI
- net PMOD_SDI: now also PMOD_OLED.2 (Pin_2); no longer U5.5 (SCL)
- removed net 33SDA: IC2.46 (IOB_0A), R18.1, U5.4 (SDA)
- new net I2C_SCL: IC2.38 (IOT_50B), PMOD_TMP2.1 (Pin_1), PMOD_TMP2.5 (Pin_5)
- new net I2C_SDA: IC2.37 (IOT_45A_G1), PMOD_TMP2.2 (Pin_2), PMOD_TMP2.6 (Pin_6)
- new net PMOD_SS: IC2.46 (IOB_0A), PMOD_OLED.1 (Pin_1)
- no-connect marks 19 -> 14
Other:
- note removed: "CE0 (SPI FPGA)"
- note removed: "CE1 (SPI FLASH)"
- note removed: "USB"
- note removed: "^"
- moved on the sheet: C15, C16, C17, C18, C45, C46, C47, C48, PMOD_OLED, Q1, R12, R15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

Commit message: Replaced FPGA
Parts:
- removed C19, C21, C23, C25, C33: 100n, symbol Device:C
- removed C20, C28, C29, C30, C31: 4.7u, symbol Device:C
- removed IC2: ICE5LP2K-SG48ITR, QFN50P700X700X100-49N-D, symbol ICE5LP2K-SG48ITR:ICE5LP2K-SG48ITR
- removed JP2: Jumper_3_Open, symbol Jumper:Jumper_3_Open
- removed PS1: TLV75733PDBVR, SOT95P280X145-5N, symbol TLV75733PDBVR:TLV75733PDBVR
- removed PS2: TLV75712PDBVR, SOT95P280X145-5N, symbol TLV75712PDBVR:TLV75712PDBVR
- removed R10: 10k, symbol Device:R
- removed R9: 100, symbol Device:R
- removed SW6: SW_Push, symbol Switch:SW_Push
- removed U2: MCP1804x-2502xOT, Package_TO_SOT_SMD:SOT-23-5, symbol Regulator_Linear:MCP1804x-2502xOT
- added C32, C56, C60: 4.7u, symbol Device:C
- added C55, C58, C61, C63: 100n, symbol Device:C
- added C57, C59: 1u, symbol Device:C
- added D7: D, symbol Device:D
- added JP1: Jumper_3_Open, symbol Jumper:Jumper_3_Open
- added R16: 10k, symbol Device:R
- added R19, R23: 3.3k, symbol Device:R
- added TP1, TP10, TP11, TP12, TP13, TP14, TP15, TP18, TP19, TP2, TP20, TP21, TP22, TP3, TP4, TP5, TP6, TP7, TP8, TP9: TestPoint, symbol Connector:TestPoint
- added U7: ICE40UP5K-SG48I, QFN48_L-ASC10_ICE40ULTRAPLUS_MACHXO2_LAT, symbol FPGA5k:ICE40UP5K-SG48I
- added U8: XC6206P122MR-G, SOT-23_TOR, symbol VREG1_2V:XC6206P122MR-G
- added U9: XC6206P332MR, SOT-23_TOR, symbol VREG3_3V:XC6206P332MR
- C1: value 1u -> 0.1
- C2: value 1u -> 4.7
- C34: value 1u -> 4.7u
- C35: value 1u -> 100n
- R13, R14, R3, R4: value 10k -> 65.7
- R15: value 0.02/ 2 W -> 0.02/ 5 W
- R17: value 10k -> 100
- R20: value 0.02 -> 0.02 5W
- R8: value 66.5 -> 65.7
Connections:
- net +1V2: now also R17.1, C63.2, U7.30 (VCC)
- net +2V5: now also C2.1, D7.1 (K), JP1.1 (A); no longer C34.1
- net +3V3: now also C32.1, C55.2, C56.1, C58.2, C60.1, C61.2, JP1.3 (B), R16.1, R19.1, R23.1, U7.1 (VCCIO_2), U7.22 (SPI_Vccio1), U7.33 (VCCIO_0); no longer C35.1, R17.1
- net +5V: now also D13.1 (K), C59.1, U8.3 (VIN), U9.3 (VIN); no longer C1.1
- net 1.2: now also C57.1, TP22.1, U8.2 (VOUT); no longer C4.1
- net 3.3: now also C1.1, C4.1, D7.2 (A), TP18.1, U9.2 (VOUT); no longer C2.1
- net B_LED: now also U7.40 (RGB1)
- net DC_PMOD: now also U7.43 (IOT_49a)
- net FPGA_CLK: now also U7.35 (IOT_46b_G0)
- net GND: now also C35.1, D13.2 (A), C32.2, C55.1, C56.2, C57.2, C58.1, C59.2, C60.2, C61.1, C63.1, U7.49, U8.1 (VSS), U9.1 (VSS); no longer C35.2
- net G_LED: now also U7.39 (RGB0)
- net I2C_SCL: now also R23.2, U7.20 (IOB_25b_G3)
- net I2C_SDA: now also R19.2, U7.21 (IOB_23b)
- net PMOD_CLK: now also U7.44 (IOB_3b_G6)
- net PMOD_SS: now also U7.46 (IOB_0a)
- net RES_PMOD: now also U7.42 (IOT_51a); no longer R8.2
- net R_LED: now also U7.41 (RGB2)
- net SCK: now also U7.15 (IOB_34a_SPI_SCK)
- net SCL: now also U7.47 (IOB_2a)
- net SDA: now also U7.48 (IOB_4a)
- net SDI: now also U7.17 (IOB_33b_SPI_SI)
- net SDO: now also U7.14 (IOB_32a_SPI_SO)
- net SD_IO2: now also TP19.1, U7.18 (IOB_31b)
- net SD_IO3: now also U7.19 (IOB_29b)
- net SS: now also U7.16 (IOB_35b_SPI_SS)
- net button1: now also U7.28 (IOT_41a)
- net button2: now also U7.27 (IOT_38b)
- net button3: now also U7.26 (IOT_39a)
- net button4: now also U7.25 (IOT_36b)
- net cdone: now also TP21.1, U7.7 (CDONE)
- net creset: now also R8.2, R16.2, TP20.1, U7.8 (creset_b); no longer R17.2
- net VDDC: now reaches PMOD_OLED.10 (Pin_10)
- net VDDC: now also U7.37 (IOT_45a_G1)
- net VBAT: now reaches PMOD_OLED.9 (Pin_9)
- net VBAT: now also U7.38 (IOT_50b)
- net at FB1.2, J1.A4 (VBUS), J1.A9 (VBUS)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: now also TP3.1
- net at J1.A8 (SBU1): now also TP1.1
- net at J1.B8 (SBU2): now also TP2.1
- net MPPTV: now reaches SW7.3
- net at U1.16 (ADBUS3): now also TP4.1
- net at U1.18 (ADBUS5): now also TP5.1
- net at U1.21 (ACBUS0): now also TP6.1
- net at U1.25 (ACBUS1): now also TP15.1
- net at U1.26 (ACBUS2): now also TP14.1
- net at U1.27 (ACBUS3): now also TP13.1
- net at U1.28 (ACBUS4): now also TP12.1
- net at U1.29 (ACBUS5): now also TP11.1
- net at U1.30 (ACBUS6): now also TP10.1
- net at U1.31 (ACBUS7): now also TP9.1
- net at U1.32 (ACBUS8): now also TP8.1
- net at U1.33 (ACBUS9): now also TP7.1
- net IOB_13B renamed OLED
- net OLED: now also U7.5 (VCC)
- net IOB_6A renamed GLED
- net GLED: now also U7.2 (IOB_6a)
- net IOB_8A renamed BLED
- net BLED: now also U7.4 (IOB_8a)
- net IOB_9B renamed RLED
- net RLED: now also U7.3 (IOB_9b)
- net PMOD_SDI renamed PMOD_SDO
- net PMOD_SDO: now also U7.45 (IOB_5b)
- new net: JP1.2 (C), U7.24 (VPP_2V5)
- new net VCC_PLL: C34.1, C35.2, R17.2, U7.29 (VCCPLL)
- no-connect marks 14 -> 16
Other:
- note added: "C2937631"
- note added: "SPI master to read configuration from FLASH at boot????"
- note removed: "C841777- shunt resistances"
- note removed: "FPGA"
- note removed: "SPI master to read configuration from FLASH at boot"
- note removed: "VBAT"
- note removed: "VDCC"
- moved on the sheet: C22461782, C36, C53, C54, C6, D13, PMOD_OLED, PMOD_TMP2, Q1, Q2, Q3, Q4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

Commit message: Modificari voltage regulator + LEDs
Parts:
- removed C57, C59: 1u, symbol Device:C
- removed D2: LD274, LED_THT:LED_D5.0mm_IRGrey, symbol LED:LD274
- removed Q1, Q2, Q3, Q4, Q5: Q_NMOS_GSD, symbol Transistor_FET:Q_NMOS_GSD
- removed R32: 162, symbol Device:R
- removed TP22: TestPoint, symbol Connector:TestPoint
- removed U8: XC6206P122MR-G, SOT-23_TOR, symbol VREG1_2V:XC6206P122MR-G
- removed U9: XC6206P332MR, SOT-23_TOR, symbol VREG3_3V:XC6206P332MR
- added C19, C20: 10u, symbol Device:C
- added C21: 4.7u, symbol Device:C
- added D8: LD274, LED_THT:LED_D5.0mm_IRGrey, symbol LED:LD274
- added J2: Conn_01x02, symbol Connector_Generic:Conn_01x02
- added J3: Conn_01x11, symbol Connector_Generic:Conn_01x11
- added J4: Conn_01x06, symbol Connector_Generic:Conn_01x06
- added L1: L, symbol Device:L
- added L2: 2.2u, symbol Device:L
- added R10: 100, symbol Device:R
- added R24: 360k, symbol Device:R
- added R9: 549, symbol Device:R
- added SW6: EG1218, SW_1218_EWI, symbol slide_sw:EG1218
- added TP16, TP17: TestPoint, symbol Connector:TestPoint
- added U2: TPS62026DRCR, DRC10_2P4X1P65, symbol Vreg3V3:TPS62026DRCR
- added U9: TPS62242DRVR, DRV6_1P6X1, symbol Vreg1.2:TPS62242DRVR
- C3: value 1u -> 22pF; JLCPCB (none) -> C466226
- C4: value 1u -> 10u; JLCPCB (none) -> C77041
- R12: value 121 -> 360k
- R29: value 121 -> 100
- R30: value 158 -> 549
- R31: value 115 -> 100
- R33: value 70 -> 549
- R34, R35: value 35 -> 50.5
- renumbered C22461782 to C5393554
Connections:
- net +3V3: now also D3.2 (A), D4.2 (A), D5.2 (A), D6.2 (A), D8.2 (A)
- net +5V: now also C19.1, U2.1 (EN), U2.2 (VIN), U2.3 (VIN); no longer C3.1, D3.2 (A), D4.2 (A), D5.2 (A), D6.2 (A)
- net 1.2: now also C3.2, C4.2, R12.2, TP18.1, L2.1
- net 3.3: now also C21.2, SW6.2, U9.4 (EN), U9.5 (VIN); no longer C4.1, TP18.1
- net BLED: now also R31.2
- net GLED: now also R29.2
- net GND: now also C4.1, C19.2, C20.2, C21.1, J4.1 (Pin_1), R24.1, U2.10 (PGND), U2.4 (GND), U2.6 (MODE), U2.9 (PGND), U9.2 (MODE), U9.6 (GND); no longer C3.2, C4.2
- net I2C_SCL: now also U7.9 (IOB_16a); no longer U7.20 (IOB_25b_G3)
- net I2C_SDA: now also U7.10 (IOB_18a); no longer U7.21 (IOB_23b)
- net MPPTV: now also J4.6 (Pin_6), SW6.1; no longer SW7.3
- net OLED: now also R9.2
- net RLED: now also R30.2
- net SCL: now also J2.1 (Pin_1)
- net SDA: now also J2.2 (Pin_2)
- net VDDC: now also U7.36 (IOT_48b); no longer U7.37 (IOT_45a_G1)
- net cdone: now also R10.2
- net at R12.1: now also C3.1, R24.2, U9.3 (FB)
- net at D6.1 (K): now also R9.1
- net IOB_20a: now reaches U7.11 (IOB_20a)
- net IOB_20a: now also J3.4 (Pin_4)
- net IOB_22a: now reaches U7.12 (IOB_22a)
- net IOB_22a: now also J3.5 (Pin_5)
- net IOB_24a: now reaches U7.13 (IOB_24a)
- net IOB_24a: now also J3.6 (Pin_6)
- net IOT_37a: now reaches U7.23 (IOT_37a)
- net IOT_37a: now also J3.7 (Pin_7)
- net IOT_42b: now reaches U7.31 (IOT_42b)
- net IOT_42b: now also J3.11 (Pin_11)
- net IOT_43a: now reaches U7.32 (IOT_43a)
- net IOT_43a: now also J3.10 (Pin_10)
- net IOT_44b: now reaches U7.34 (IOT_44b)
- net IOT_44b: now also J3.9 (Pin_9)
- net IOB_13b: now reaches U7.6 (IOB_13b)
- net IOB_13b: now also J3.1 (Pin_1)
- new net: C20.1, L1.2, SW6.3, TP16.1, U2.5 (FB)
- new net: L2.2, U9.1 (SW)
- new net: TP17.1, U9.7 (EPAD)
- new net: D8.1 (K), R10.1
- new net: L1.1, U2.7 (SW), U2.8 (SW)
- new net CE: J4.5 (Pin_5)
- new net INT: J4.4 (Pin_4)
- new net IOB_23b: J3.3 (Pin_3), U7.21 (IOB_23b)
- new net IOB_25b_G3: J3.2 (Pin_2), U7.20 (IOB_25b_G3)
- new net IOT_45a_G1: J3.8 (Pin_8), U7.37 (IOT_45a_G1)
- new net SCL_HOST: J4.2 (Pin_2)
- new net SDA_HOST: J4.3 (Pin_3)
- no-connect marks 16 -> 6
Other:
- note added: "0.6A"
- note added: "BLUE C5354973"
- note added: "GREEN C5875752"
- note added: "ORANGE C5588281"
- note added: "RED C5366382"
- note removed: "BLUE C965807"
- note removed: "GREEN C965804"
- note removed: "ORANGE C965800"
- note removed: "RED C965799"
- moved on the sheet: C1, C11, C12, C13, C14, C15, C16, C17, C18, C2, C26, C45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

Commit message: Added external connectors
Parts:
- removed J3: Conn_01x11, symbol Connector_Generic:Conn_01x11
- added J5, J6, J7: Conn_01x02, symbol Connector_Generic:Conn_01x02
- added J8: Conn_01x10, symbol Connector_Generic:Conn_01x10
Connections:
- net IOB_13b is gone; now on net OLED: U7.6 (IOB_13b)
- net +1V2: now also U7.5 (VCC)
- net +3V3: now also J6.2 (Pin_2), J7.2 (Pin_2)
- net +5V: now also J5.2 (Pin_2)
- net GND: now also J5.1 (Pin_1), J6.1 (Pin_1), J7.1 (Pin_1)
- net IOB_20a: now also J8.1 (Pin_1)
- net IOB_22a: now also J8.2 (Pin_2)
- net IOB_23b: now also J8.5 (Pin_5)
- net IOB_24a: now also J8.3 (Pin_3)
- net IOB_25b_G3: now also J8.4 (Pin_4)
- net IOT_37a: now also J8.6 (Pin_6)
- net IOT_42b: now also J8.10 (Pin_10)
- net IOT_43a: now also J8.9 (Pin_9)
- net IOT_44b: now also J8.8 (Pin_8)
- net IOT_45a_G1: now also J8.7 (Pin_7)
- net OLED: no longer U7.5 (VCC)
Other:
- note added: "external connectors"
- moved on the sheet: J2, J4

Commit message: Footprints added
Parts:
- removed C1: 0.1, symbol Device:C
- removed C10: C_Polarized, symbol Device:C_Polarized
- removed C11, C12, C13, C14, C15, C16, C17, C18, C22, C24, C26, C35, C36, C37, C38, C39, C40, C42, C44, C5, C53, C55, C58, C6, C61, C63, C7, C8, C9: 100n, symbol Device:C
- removed C19, C20, C4: 10u, symbol Device:C
- removed C2: 4.7, symbol Device:C
- removed C21, C27, C32, C34, C41, C43, C54, C56, C60: 4.7u, symbol Device:C
- removed C3: 22pF, symbol Device:C
- removed C45, C46, C47, C49, C50, C51: 47u, symbol Device:C
- removed C48, C52: 0.1u, symbol Device:C
- removed D1: LED, symbol Device:LED
- removed D3: LD274, LED_THT:LED_D5.0mm_IRGrey, symbol LED:LD274
- removed FB1, FB3, FB4: FerriteBead, symbol Device:FerriteBead
- removed IC1: AT25FF081A-SSHN-B, SOIC127P600X175-8N, symbol AT25FF081A-SSHN-B:AT25FF081A-SSHN-B
- removed J7: Conn_01x02, symbol Connector_Generic:Conn_01x02
- removed L2: 2.2u, symbol Device:L
- removed R1, R16, R2, R21, R25, R28: 10k, symbol Device:R
- removed R10, R17, R31: 100, symbol Device:R
- removed R11, R18: 3.3k, symbol Device:R
- removed R12: 360k, symbol Device:R
- removed R15: 0.02/ 5 W, symbol Device:R
- removed R20: 0.02 5W, symbol Device:R
- removed R22: 12k, symbol Device:R
- removed R33: 549, symbol Device:R
- removed R35: 50.5, symbol Device:R
- removed R5, R6: 5.1k, symbol Device:R
- removed R7: 121, symbol Device:R
- removed R8: 65.7, symbol Device:R
- removed TP19: TestPoint, symbol Connector:TestPoint
- removed U9: TPS62242DRVR, DRV6_1P6X1, symbol Vreg1.2:TPS62242DRVR
- added C1, C10, C11, C12, C13, C14, C15, C16, C17, C18, C23, C24, C25, C26, C27, C28, C29, C30, C35, C37, C38, C39, C46, C48, C50, C52, C55, C57, C6, C7, C8, C9: 100nF, PCM_JLCPCB:C_0603, symbol PCM_JLCPCB-Capacitors:0603,100nF
- added C19, C36: 10u, EasyEDA:C1206, symbol Cap10u:JMK316BJ106KL-T
- added C2, C22, C31, C32, C33, C34, C47, C49, C51, C53, C56: 4.7uF, PCM_JLCPCB:C_0603, symbol PCM_JLCPCB-Capacitors:0603,4.7uF
- added C20, C3: 4.7u, EasyEDA:C0603, symbol Cap4_7u:GRM188R60J475KE19D
- added C21: 10u, EasyEDA:C0603, symbol Cap10u_murata:GRM188R60J106ME47D
- added C4: 22pF, PCM_JLCPCB:C_0603, symbol PCM_JLCPCB-Capacitors:0603,22pF
- added C40, C41, C42, C43, C44, C45, C5: 47uF, PCM_JLCPCB:C_1206, symbol PCM_JLCPCB-Capacitors:1206,47uF
- added D1: LD274, EasyEDA:LED-SMD_L1.0-W0.5-RD, symbol LED:LD274
- added D2: LD274, LED_THT:LED_D5.0mm_IRGrey, symbol LED:LD274
- added J3: Conn_01x02, Connector_PinHeader_2.54mm:PinHeader_1x02_P2.54mm_Vertical, symbol Connector_Generic:Conn_01x02
- added L3: GZ1608D601TF, EasyEDA:L0603, symbol FerriteBead:GZ1608D601TF
- added L4, L5: BLM18HE152SN1D, EasyEDA:L0603, symbol FB_FTDI:BLM18HE152SN1D
- added L6: 2.2u, EasyEDA:IND-SMD_L3.0-W3.0_LPS3015-222ML, symbol L_2_2u:LPS3015-222MRC
- added R1, R2: 5.1kΩ, PCM_JLCPCB:R_0603, symbol PCM_JLCPCB-Resistors:0603,5.1kΩ
- added R10: 560Ω, PCM_JLCPCB:R_0603, symbol PCM_JLCPCB-Resistors:0603,560Ω
- added R11: 2.2kΩ, PCM_JLCPCB:R_0603, symbol PCM_JLCPCB-Resistors:0603,2.2kΩ
- added R12, R17: 360kΩ, PCM_JLCPCB:R_0603, symbol PCM_JLCPCB-Resistors:0603,360kΩ
- added R15, R16, R18, R20, R26, R32, R36, R37, R8: 10kΩ, PCM_JLCPCB:R_0603, symbol PCM_JLCPCB-Resistors:0603,10kΩ
- added R21: 100Ω, PCM_JLCPCB:R_0603, symbol PCM_JLCPCB-Resistors:0603,100Ω
- added R22, R7: 3.3kΩ, PCM_JLCPCB:R_0603, symbol PCM_JLCPCB-Resistors:0603,3.3kΩ
- added R25: 750Ω, PCM_JLCPCB:R_0603, symbol PCM_JLCPCB-Resistors:0603,750Ω
- added R5: 12kΩ, PCM_JLCPCB:R_0603, symbol PCM_JLCPCB-Resistors:0603,12kΩ
- added R6: 1.4k, EasyEDA:R0603, symbol 1.4k:0603WAF1401T5E
- added U10, U11: 20m, EasyEDA:RES-SMD_L7.1-W4.6_HOXLR2818, symbol R20m:HOXLR2818-5W-20MR-1%
- added U12: TPS62240DRVR, DRV6_1P6X1, symbol Vreg1v2:TPS62240DRVR
- added U8: W25Q32JVSSIQ, EasyEDA:SOIC-8_L5.3-W5.3-P1.27-LS8.0-BL, symbol FLASH:W25Q32JVSSIQ
- C5393554: footprint (none) -> EasyEDA:LED-SMD_4P-L3.0-W1.5_APFA3010LSEEZGKQBKC; JLCPCB (none) -> C5393554
- D13: JLPCPCB (none) -> C110760
- D4: footprint LED_THT:LED_D5.0mm_IRGrey -> PCM_JLCPCB:D_0805; JLCPCB (none) -> C5366382
- D5: footprint LED_THT:LED_D5.0mm_IRGrey -> EasyEDA:LED-SMD_L1.0-W0.5-RD; JLCPCB (none) -> C5354973
- D6: footprint LED_THT:LED_D5.0mm_IRGrey -> EasyEDA:LED-SMD_L2.1-W1.0-FD_UMD960; JLCPCB (none) -> C5588281
- D7: footprint (none) -> EasyEDA:SOD-523_L1.2-W0.8-LS1.6-RD; JLCPCB (none) -> C727112
- D8: JLCPCB (none) -> C5875752
- J2, J5, J6: footprint (none) -> Connector_PinHeader_2.54mm:PinHeader_1x02_P2.54mm_Vertical; JLCPB (none) -> C32713268
- J4: footprint (none) -> Connector_PinHeader_2.54mm:PinHeader_1x06_P2.54mm_Vertical; JLCPCB (none) -> C56816
- J8: footprint (none) -> EasyEDA:HDR-TH_10P-P2.00-V-F; JLCPCB (none) -> C69515
- L1: value L -> 10u; footprint (none) -> Inductor_SMD:L_APV_ANR6045; JLCPCB (none) -> C5259068
- PMOD_OLED: footprint (none) -> Connector_PinSocket_2.00mm:PinSocket_2x06_P2.00mm_Horizontal; JLCPCB (none) -> C5333437
- PMOD_TMP2: footprint (none) -> Connector_PinHeader_2.54mm:PinHeader_2x04_P2.54mm_Horizontal; JLCPCB (none) -> C7529541
- R24: value 360k -> 549; footprint (none) -> PCM_JLCPCB:R_0603; JLCPCB (none) -> C13007
- R27: value 2.2k -> 324; JLCPCB (none) -> C12963
- R29: value 100 -> 549; footprint (none) -> PCM_JLCPCB:R_0603; JLCPCB (none) -> C13007
- R30, R9: value 549 -> 909; footprint (none) -> PCM_JLCPCB:R_0603; JLCPCB (none) -> C13050
- R34: value 50.5 -> 324; JLCPCB (none) -> C12963
- SW3: footprint (none) -> EasyEDA:SW-TH_4P-L6.0-W6.0-P4.50-LS6.5; JLCPCB (none) -> C455095
- SW6, SW7: JLCPCB (none) -> C273394
- U3: JLCPCB (none) -> C2862074
- XTAL1: JLCPCB (none) -> C596950
Connections:
- net +1V2: now also J6.2 (Pin_2), C40.1, C41.1, C42.1, C47.1, C48.1, C49.1, C50.1, R21.2, U10.1
- net +2V5: now also C2.1
- net +3V3: now also C23.1, C3.1, C32.1, C38.1, C39.1, C43.1, C44.1, C45.1, C51.1, C52.1, C53.1, C55.1, C6.1, D1.2 (A), J3.2 (Pin_2), R16.1, R22.1, R26.1, R32.1, R36.1, R37.1, R7.1, R8.1, U11.1, U8.8 (VCC); no longer J6.2 (Pin_2), U1.34 (RESET#), U6.6 (VCC)
- net +5V: now also C19.2, C22.1, C5.1, D2.2 (A)
- net 1.2: now also C15.1, C16.1, C17.1, C18.1, C21.1, C4.1, L6.1, R17.1, U10.2
- net 3.3: now also U1.34 (RESET#), U1.39 (VCCD), U6.6 (VCC), C1.1, C11.1, C12.1, C13.1, C14.1, C20.1, C25.1, C26.1, C27.1, C28.1, C46.1, C7.1, C8.1, C9.1, L4.1, L5.1, R15.1, R18.1, R20.1, U11.2, U12.4 (EN), U12.5 (VIN)
- net BLED: now also R24.2
- net B_LED: now also R27.2
- net EE_CLK: now also R20.2
- net EE_CS: now also R18.2
- net EE_DAT: now also R11.1; no longer R27.1
- net FT_VCORE: now also C37.1
- net GND: now also C1.2, C10.2, C11.2, C12.2, C13.2, C14.2, C15.2, C16.2, C17.2, C18.2, C19.1, C2.2, C20.2, C21.2, C22.2, C23.2, C24.2, C25.2, C26.2, C27.2, C28.2, C29.2, C3.2, C30.2, C31.2, C32.2, C33.2, C34.2, C35.2, C36.1, C37.2, C38.2, C39.2, C40.2, C41.2, C42.2, C43.2, C44.2, C45.2, C46.2, C47.2, C48.2, C49.2, C5.2, C50.2, C51.2, C52.2, C53.2, C55.2, C56.2, C57.2, C6.2, C7.2, C8.2, C9.2, J3.1 (Pin_1), R1.2, R12.2, R2.2, R5.1, R6.1, U12.2 (MODE), U12.6 (GND), U8.4 (GND); no longer R24.1
- net R_LED: now also R25.2
- net SCK: now also R26.2, U8.6 (CLK)
- net SCL: now also R22.2
- net SDA: now also R7.2
- net SDI: now also U8.2 (DO（IO1）)
- net SDO: now also U8.5 (DI（IO0）)
- net SD_IO2: now also R36.2, U8.3 (IO2)
- net SD_IO3: now also R32.2, U8.7 (IO3)
- net SS: now also R37.2, U8.1 (~{CS})
- net VCC_PLL: now also C34.1, C35.1, R21.1
- net VPHY: now also C29.1, C31.1, L4.2
- net VPLL: now also C30.1, C33.1, L5.2
- net cdone: now also R10.2
- net creset: now also R16.2, R8.2
- net at SW7.1: now also C10.1, L3.2
- net at J1.A4 (VBUS), J1.A9 (VBUS), J1.B4 (VBUS)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: now also L3.1
- net at L1.2, SW6.3, TP16.1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: now also C36.2
- net at J1.A5 (CC1): now also R1.1
- net at J1.B5 (CC2): now also R2.1
- net at U6.1 (DO): now also R11.2, R15.2; no longer R27.2
- net at R29.1: now also D1.1 (K)
- net at TP17.1: now also U12.7 (EPAD)
- net at D8.1 (K): now also R10.1
- net at C5393554.3 (BK): now also R27.1
- net at D5.1 (K): now also R24.1
- net at U1.37 (VCCA): now also C24.1
- net at C5393554.2 (RK): now also R25.1
- net at U1.5 (REF): now also R5.2
- net at JP1.2 (C), U7.24 (VPP_2V5): now also C56.1, C57.1
- new net: L6.2, U12.1 (SW)
- new net: C4.2, R12.1, R17.2, U12.3 (FB)
- new net: D2.1 (K), R6.2
- no-connect marks 6 -> 5
Other:
- note added: "BLUE"
- note added: "EEPROM"
- note added: "EXTERNAL CONNECTORS"
- note added: "FPGA"
- note added: "FTDI"
- note added: "GREEN"
- note added: "ORANGE"
- note added: "POWER MEASUREMENT"
- note added: "RED"
- note added: "VOLTAGE REGULATORS"
- note removed: "8Mbit"
- note removed: "BLUE C5354973"
- note removed: "C2937631"
- note removed: "ORANGE C5588281"
- note removed: "RED C5366382"
- note removed: "SPI master to read configuration from FLASH at boot????"
- note removed: "external connectors"
- note removed: "pullup on ss means configure as"
- moved on the sheet: C5393554, D13, D7, J2, J4, J8, JP1, L1, PMOD_OLED, PMOD_TMP2, R13, R14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
