File: First_try.kicad_sch (KiCad schematic)
At the start: 139 parts, among them J1 TYPE-611-T3-W, J11 Conn_01x20, J2 Conn_01x02, J3 Conn_01x02, J4 Conn_01x06, J5 Conn_01x02, J6 Conn_01x02, J7 Conn_01x02, J9 Conn_01x20, SW1 SW_Push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

Commit message: Layout modifications
Parts:
- removed J11, J9: Conn_01x20, Connector_PinHeader_2.54mm:PinHeader_1x20_P2.54mm_Vertical, symbol Connector_Generic:Conn_01x20
- removed J4: Conn_01x06, Connector_PinHeader_2.54mm:PinHeader_1x06_P2.54mm_Vertical, symbol Connector_Generic:Conn_01x06
- removed SW6: EG1218, footprints:SW_1218_EWI, symbol slide_sw:EG1218
- removed TP1, TP2: TestPoint, TestPoint:TestPoint_Pad_1.0x1.0mm, symbol Connector:TestPoint
- added J10, J4: Conn_01x11, Connector_PinHeader_2.54mm:PinHeader_1x11_P2.54mm_Vertical, symbol Connector_Generic:Conn_01x11
- added J9: Conn_01x02, Connector_PinHeader_2.54mm:PinHeader_1x02_P2.54mm_Vertical, symbol Connector_Generic:Conn_01x02
Connections:
- net IOB_23b is gone; now on net GLED: U7.21 (IOB_23b)
- net IOB_25b_G3 is gone; now on net FPGA_CLK: U7.20 (IOB_25b_G3)
- net IOT_36b is gone; now on net SCL: U7.25 (IOT_36b)
- net IOT_37a is gone; now on net BLED: U7.23 (IOT_37a)
- net IOT_38b is gone; now on net PMOD_CLK: U7.27 (IOT_38b)
- net IOT_39a is gone; now on net SDA: U7.26 (IOT_39a)
- net IOT_41a is gone; now on net VDDC: U7.28 (IOT_41a)
- net IOT_42b is gone; now on net VBAT: U7.31 (IOT_42b)
- net IOT_43a is gone; now on net PMOD_SDO: U7.32 (IOT_43a)
- net IOT_44b is gone; now on net RES_PMOD: U7.34 (IOT_44b)
- net IOT_45a_G1 is gone; now on net button1: U7.37 (IOT_45a_G1)
- net +1V2: now also J10.10 (Pin_10), J10.11 (Pin_11), J10.9 (Pin_9)
- net +3V3: now also J10.4 (Pin_4), J10.5 (Pin_5), J10.6 (Pin_6)
- net +5V: now also J10.1 (Pin_1), J10.2 (Pin_2), J10.3 (Pin_3); no longer U1.40 (VREG)
- net 3.3: now also C36.2, L1.1, TP16.1, U1.40 (VREG), U2.5 (FB)
- net BLED: no longer U7.4 (IOB_8a)
- net DC_PMOD: now also U7.36 (IOT_48b); no longer U7.43 (IOT_49a)
- net FPGA_CLK: no longer U7.35 (IOT_46b_G0)
- net GLED: no longer U7.2 (IOB_6a)
- net GND: now also J10.7 (Pin_7), J10.8 (Pin_8)
- net I2C_SCL: now also U7.13 (IOB_24a); no longer U7.9 (IOB_16a)
- net I2C_SDA: now also U7.12 (IOB_22a); no longer U7.10 (IOB_18a)
- net OLED: now also U7.43 (IOT_49a); no longer U7.6 (IOB_13b)
- net PMOD_CLK: no longer U7.44 (IOB_3b_G6)
- net PMOD_SDO: no longer U7.45 (IOB_5b)
- net PMOD_SS: no longer U7.46 (IOB_0a)
- net RES_PMOD: no longer U7.42 (IOT_51a)
- net RLED: now also U7.38 (IOT_50b); no longer U7.3 (IOB_9b)
- net SCL: now also J2.2 (Pin_2); no longer U7.47 (IOB_2a)
- net SDA: now also J9.1 (Pin_1), J9.2 (Pin_2); no longer J2.2 (Pin_2), U7.48 (IOB_4a)
- net SD_IO2: now also U7.19 (IOB_29b); no longer U7.18 (IOB_31b)
- net SD_IO3: now also U7.18 (IOB_31b); no longer U7.19 (IOB_29b)
- net VBAT: no longer U7.38 (IOT_50b)
- net VDDC: no longer U7.36 (IOT_48b)
- net button1: no longer U7.11 (IOB_20a)
- net button2: now also U7.42 (IOT_51a); no longer U7.12 (IOB_22a)
- net button3: now also U7.44 (IOB_3b_G6); no longer U7.13 (IOB_24a)
- new net PIN1: J4.1 (Pin_1), U7.11 (IOB_20a)
- new net PIN10: J4.10 (Pin_10), U7.46 (IOB_0a)
- new net PIN11: J4.11 (Pin_11), U7.45 (IOB_5b)
- new net PIN2: J4.2 (Pin_2), U7.10 (IOB_18a)
- new net PIN3: J4.3 (Pin_3), U7.9 (IOB_16a)
- new net PIN4: J4.4 (Pin_4), U7.6 (IOB_13b)
- new net PIN5: J4.5 (Pin_5), U7.4 (IOB_8a)
- new net PIN6: J4.6 (Pin_6), U7.3 (IOB_9b)
- new net PIN7: J4.7 (Pin_7), U7.2 (IOB_6a)
- new net PIN8: J4.8 (Pin_8), U7.48 (IOB_4a)
- new net PIN9: J4.9 (Pin_9), U7.47 (IOB_2a)
- no-connect marks 5 -> 7
Other:
- moved on the sheet: PMOD_TMP2, R19, R23

Commit message: Last version
Parts:
- C19, C36: LCSC (none) -> C92789
- C20, C3: LCSC (none) -> C71631
- C21: LCSC (none) -> C77041
- C5393554: LCSC (none) -> C5393554
- D1, D2: LCSC (none) -> C5875752
- D13: LCSC (none) -> C110760
- D3: footprint LED-SMD_L1.0-W0.5-RD -> footprints:LED-SMD_L1.0-W0.5-RD; LCSC (none) -> C5875752
- D4: LCSC (none) -> C5366382
- D5: LCSC (none) -> C5354973
- D6: LCSC (none) -> C5588281
- D7: LCSC (none) -> C727112
- J1: footprint footprints:C_conn -> Connector_USB:USB_C_Receptacle_HCTL_HC-TYPE-C-16P-01A; LCSC (none) -> C2689844
- J2, J3, J5, J6, J7, J9: LCSC (none) -> C32713268
- JP1: LCSC (none) -> C24980
- L1: LCSC (none) -> C5259068
- L2, L4: LCSC (none) -> C82155
- L3: LCSC (none) -> C1002
- L6: LCSC (none) -> C2844756
- OSC1: renamed from XTAL1; value ASE-12.000MHZ-LC-T -> OSC; LCSC (none) -> C596950
- PMOD_OLED1: footprint Connector_PinSocket_2.54mm:PinSocket_2x06_P2.54mm_Horizontal -> footprints:PinSocket_2x06_P2.54mm_Horizontal_edit; LCSC (none) -> C5333437
- PMOD_TMP2: footprint Connector_PinSocket_2.54mm:PinSocket_2x04_P2.54mm_Horizontal -> footprints:PinSocket_2x04_P2.54mm_Horizontal_edit; LCSC (none) -> C7529541
- R6: LCSC (none) -> C25957
- SW1, SW2, SW3, SW4: LCSC (none) -> C455095
- SW7: LCSC (none) -> C273394
- U1: LCSC (none) -> C51997
- U10, U11: LCSC (none) -> C4944045
- U12: LCSC (none) -> C398345
- U2: LCSC (none) -> C2071183
- U3: LCSC (none) -> C2862074
- U4, U5: LCSC (none) -> C49851
- U6: LCSC (none) -> C190271
- U8: LCSC (none) -> C82344
Connections:
- net PMOD_SS: now also U7.35 (IOT_46b_G0)

Commit message: RISC-V added
Other:
- note added: "active low"
Changed lines of the file:
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@@
 		)
 	)
+	(text "active low"
+		(exclude_from_sim no)
+		(at 280.416 152.146 0)
+		(effects
+			(font
+				(size 1.27 1.27)
+			)
+		)
+	)
 	(text "FLASH\n"
 		(exclude_from_sim no)
@@
 		(dnp no)
 		(property "Reference" "L3"
-			(at 73.533 44.958 0)
+			(at 75.438 51.308 0)
 			(effects
 				(font
@@
 		)
 		(property "Value" "GZ1608D601TF"
-			(at 73.66 47.244 0)
+			(at 74.422 46.99 0)
 			(effects
 				(font
@@
 		(on_board yes)
 		(dnp no)
-		(fields_autoplaced yes)
 		(property "Reference" "TP3"
 			(at 66.04 44.9579 0)
@@
 		)
 		(property "Value" "TestPoint"
-			(at 66.04 47.4979 0)
+			(at 62.992 51.816 0)
 			(effects
 				(font
